File: Libra mini EC.kicad_pcb (KiCad board)
At the start: 2 copper layers, 27.5 x 104 mm, 142 parts, among them J1 USB_C_Receptacle_USB2.0_16P, J3 Conn_01x18, J4 Conn_01x18, SW1 EC_SW, SW10 EC_SW, SW11 EC_SW, SW12 EC_SW, SW13 EC_SW, SW14 EC_SW, SW15 EC_SW, SW16 EC_SW, SW17 EC_SW, SW18 EC_SW, SW19 EC_SW, SW2 EC_SW, SW20 EC_SW, SW21 EC_SW, SW22 EC_SW, SW23 EC_SW, SW24 EC_SW, SW25 EC_SW, SW26 EC_SW, SW27 EC_SW, SW28 EC_SW, SW29 EC_SW, SW3 EC_SW, SW30 EC_SW, SW31 EC_SW, SW32 EC_SW, SW33 EC_SW, SW34 EC_SW, SW35 EC_SW, SW36 EC_SW, SW37 EC_SW, SW38 EC_SW, SW39 EC_SW, SW4 EC_SW, SW40 EC_SW, SW41 EC_SW, SW42 EC_SW, SW43 EC_SW, SW44 EC_SW, SW45 EC_SW, SW46 EC_SW, SW47 EC_SW, SW5 EC_SW, SW6 EC_SW, SW7 EC_SW, SW8 EC_SW, SW9 EC_SW, U1 STM32G474CBTx, U2 USBLC6-2SC6, U3 TPS7A2033, U4 TPS7A2033, U5 TPS7A2033, U6 OPA2365, U7 4052, U8 OPA2365, U9 4052, Y1 8Mhz 12pF

Commit message: 14.04.2026
Parts:
- removed SW44: EC_SW, Kicad footprints:ecs_pad_1U_hybrid_hotswap_V2
- added SW48: EC_SW, Kicad footprints:ecs_pad_hybrid hotswap_1.25-1_libra_2.286, F.Cu at (204.6, 82.0)
- BOOT_SW1, RESET_SW1: value SW_MEC_5G -> Omron b3u
- SW45: footprint Kicad footprints:ecs_pad_1U_hybrid_hotswap_V2 -> Kicad footprints:ecs_pad_hybrid_hotswap_1.25-1_libra_7.239
- SW46: footprint Kicad footprints:ecs_pad_1U_hybrid_hotswap_V2 -> Kicad footprints:ecs_pad_hybrid_hotswap_1.25-1_libra_2.381
- U4, U6, U7, U8, U9: moved to B.Cu
- moved U4 46.6 mm to (368.7, 54.6), turned to -90 degrees
- moved U7 23.3 mm to (373.3, 65.4), turned to -90 degrees
- moved BOOT_SW1 21.0 mm to (349.7, 56.0)
- moved RESET_SW1 21.0 mm to (349.7, 60.4)
- moved U8 9.12 mm to (350.9, 80.0), turned to 180 degrees
- moved U6 8.45 mm to (362.4, 65.3), turned to -90 degrees
- moved U9 8.07 mm to (359.5, 79.9), turned to 180 degrees
- moved U5 7.28 mm to (332.2, 93.5)
- moved SW8 0.66 mm to (179.2, 28.5)
- moved SW10 0.66 mm to (216.9, 23.2)
- moved SW20 0.66 mm to (166.2, 49.3)
- moved SW21 0.66 mm to (185.0, 46.6)
- moved SW22 0.66 mm to (203.9, 44.0)
- moved SW7 0.66 mm to (160.3, 31.2)
- moved SW9 0.66 mm to (198.1, 25.9)
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Connections:
- BOOT_SW1 pad 2: BOOT0 -> +3.3V
- RESET_SW1 pad 2: RESET -> GND
Other:
- board size 27.5 x 104 mm -> 403.9 x 104 mm
