File: Libra mini EC.kicad_pcb (KiCad board)
At the start: 2 copper layers, 403.9 x 104 mm, 142 parts, among them J1 USB_C_Receptacle_USB2.0_16P, J3 Conn_01x18, J4 Conn_01x18, SW1 EC_SW, SW10 EC_SW, SW11 EC_SW, SW12 EC_SW, SW13 EC_SW, SW14 EC_SW, SW15 EC_SW, SW16 EC_SW, SW17 EC_SW, SW18 EC_SW, SW19 EC_SW, SW2 EC_SW, SW20 EC_SW, SW21 EC_SW, SW22 EC_SW, SW23 EC_SW, SW24 EC_SW, SW25 EC_SW, SW26 EC_SW, SW27 EC_SW, SW28 EC_SW, SW29 EC_SW, SW3 EC_SW, SW30 EC_SW, SW31 EC_SW, SW32 EC_SW, SW33 EC_SW, SW34 EC_SW, SW35 EC_SW, SW36 EC_SW, SW37 EC_SW, SW38 EC_SW, SW39 EC_SW, SW4 EC_SW, SW40 EC_SW, SW41 EC_SW, SW42 EC_SW, SW43 EC_SW, SW45 EC_SW, SW46 EC_SW, SW47 EC_SW, SW48 EC_SW, SW5 EC_SW, SW6 EC_SW, SW7 EC_SW, SW8 EC_SW, SW9 EC_SW, U1 STM32G474CBTx, U2 USBLC6-2SC6, U3 TPS7A2033, U4 TPS7A2033, U5 TPS7A2033, U6 OPA2365, U7 4052, U8 OPA2365, U9 4052, Y1 8Mhz 12pF

Commit message: 14.04.2026
Parts:
- removed D13, D14: SK6812MINI, LED_SMD:LED_SK6812MINI_PLCC4_3.5x3.5mm_P1.75mm
- added REF**: MountingHole_2.2mm_M2_DIN965_Pad, MountingHole:MountingHole_2.2mm_M2_DIN965_Pad, F.Cu at (219.5, 95.9)
- added REF**: MountingHole_2.2mm_M2_DIN965_Pad, MountingHole:MountingHole_2.2mm_M2_DIN965_Pad, F.Cu at (243.5, 95.9)
- added REF**: MountingHole_2.2mm_M2_DIN965_Pad, MountingHole:MountingHole_2.2mm_M2_DIN965_Pad, F.Cu at (243.5, 71.9)
- added REF**: MountingHole_2.2mm_M2_DIN965_Pad, MountingHole:MountingHole_2.2mm_M2_DIN965_Pad, F.Cu at (219.5, 71.9)
- added S47: MX_stab, PCM_marbastlib-mx:STAB_MX_2u, F.Cu at (265.1, 21.8)
- moved J1 280.8 mm to (142.9, 119.8)
- moved U1 280.8 mm to (142.9, 134.8)
- moved J3 202.9 mm to (134.2, 167.9), turned to -90 degrees
- moved J4 182.1 mm to (151.7, 167.2), turned to 90 degrees
- moved U9 19.1 mm to (378.2, 76.2), turned to -90 degrees
- moved U8 16.7 mm to (367.1, 75.8)
- moved C24 13.8 mm to (370.8, 81.4)
- turned SW12 to 180 degrees
- turned SW13 to 180 degrees
Connections:
- D1 pad 2: GND -> Net-(D1-VSS)
- D10 pad 2: Net-(D10-VSS) -> GND
- D11 pad 2: Net-(D10-VSS) -> GND
- D12 pad 1: Net-(D12-DOUT) -> RGB_FINISH
- D12 pad 2: Net-(D10-VSS) -> GND
- D2 pad 2: GND -> Net-(D1-VSS)
- D3 pad 2: GND -> Net-(D1-VSS)
- D4 pad 2: GND -> Net-(D1-VSS)
- D5 pad 2: GND -> Net-(D1-VSS)
- D6 pad 1: Net-(D6-DOUT) -> RGB
- D6 pad 2: GND -> Net-(D1-VSS)
- D7 pad 1: RGB -> Net-(D7-DOUT)
- D7 pad 3: Net-(D6-DOUT) -> RGB
- D8 pad 1: unconnected-(D8-DOUT-Pad1) -> Net-(D8-DOUT)
- D8 pad 2: Net-(D10-VSS) -> GND
- D8 pad 3: RGB -> Net-(D7-DOUT)
- D9 pad 2: Net-(D10-VSS) -> GND
- D9 pad 3: unconnected-(D9-DIN-Pad3) -> Net-(D8-DOUT)
Other:
- board size 403.9 x 104 mm -> 273.8 x 207.5 mm
