File: Libra mini EC.kicad_pcb (KiCad board)
At the start: 2 copper layers, 273.8 x 207.5 mm, 145 parts, among them J1 USB_C_Receptacle_USB2.0_16P, J3 Conn_01x18, J4 Conn_01x18, SW1 EC_SW, SW10 EC_SW, SW11 EC_SW, SW12 EC_SW, SW13 EC_SW, SW14 EC_SW, SW15 EC_SW, SW16 EC_SW, SW17 EC_SW, SW18 EC_SW, SW19 EC_SW, SW2 EC_SW, SW20 EC_SW, SW21 EC_SW, SW22 EC_SW, SW23 EC_SW, SW24 EC_SW, SW25 EC_SW, SW26 EC_SW, SW27 EC_SW, SW28 EC_SW, SW29 EC_SW, SW3 EC_SW, SW30 EC_SW, SW31 EC_SW, SW32 EC_SW, SW33 EC_SW, SW34 EC_SW, SW35 EC_SW, SW36 EC_SW, SW37 EC_SW, SW38 EC_SW, SW39 EC_SW, SW4 EC_SW, SW40 EC_SW, SW41 EC_SW, SW42 EC_SW, SW43 EC_SW, SW45 EC_SW, SW46 EC_SW, SW47 EC_SW, SW48 EC_SW, SW5 EC_SW, SW6 EC_SW, SW7 EC_SW, SW8 EC_SW, SW9 EC_SW, U1 STM32G474CBTx, U2 USBLC6-2SC6, U3 TPS7A2033, U4 TPS7A2033, U5 TPS7A2033, U6 OPA2365, U7 4052, U8 OPA2365, U9 4052, Y1 8Mhz 12pF

Commit message: 14.04.2026
Parts:
- added J2: Conn_01x08, Kicad footprints:SOICbite_footprint, F.Cu at (337.1, 66.6)
- added SW44: EC_SW, Kicad footprints:ecs_pad_1U_hybrid_hotswap_V2, F.Cu at (226.0, 154.8)
- added SW49: EC_SW, Kicad footprints:ecs_pad_1U_hybrid_hotswap_V2, F.Cu at (226.0, 175.0)
- added SW50: EC_SW, Kicad footprints:ecs_pad_1U_hybrid_hotswap_V2, F.Cu at (226.0, 195.1)
