File: Libra mini EC.kicad_pcb (KiCad board)
At the start: 2 copper layers, 269.5 x 183.8 mm, 144 parts, among them J1 USB_C_Receptacle_USB2.0_16P, J2 Conn_01x08, J3 Conn_01x18, J4 Conn_01x18, SW1 EC_SW, SW10 EC_SW, SW11 EC_SW, SW12 EC_SW, SW13 EC_SW, SW14 EC_SW, SW15 EC_SW, SW16 EC_SW, SW17 EC_SW, SW18 EC_SW, SW19 EC_SW, SW2 EC_SW, SW20 EC_SW, SW21 EC_SW, SW22 EC_SW, SW23 EC_SW, SW24 EC_SW, SW25 EC_SW, SW26 EC_SW, SW27 EC_SW, SW28 EC_SW, SW29 EC_SW, SW3 EC_SW, SW30 EC_SW, SW31 EC_SW, SW32 EC_SW, SW33 EC_SW, SW34 EC_SW, SW35 EC_SW, SW36 EC_SW, SW37 EC_SW, SW38 EC_SW, SW39 EC_SW, SW4 EC_SW, SW40 EC_SW, SW47 EC_SW, SW5 EC_SW, SW50 EC_SW, SW51 EC_SW, SW52 EC_SW, SW53 EC_SW, SW54 EC_SW, SW55 EC_SW, SW6 EC_SW, SW7 EC_SW, SW8 EC_SW, SW9 EC_SW, U1 STM32G474CBTx, U2 USBLC6-2SC6, U3 TPS7A2033, U4 TPS7A2033, U5 TPS7A2033, U6 OPA2365, U7 4052, U8 OPA2365, U9 4052, Y1 8Mhz 12pF

Commit message: 14.04.2026
Parts:
- SW54, SW55: footprint Kicad footprints:ecs_pad_hybrid_hotswap_1.810 -> My_footprints:ecs_pad_hybrid_hotswap_1.25-1_libra_2.381
- moved SW54 1.13 mm to (243.6, 79.5)
- moved SW55 1.13 mm to (267.4, 79.5)
- moved S47 0.80 mm to (259.4, 22.4)
- moved SW47 0.80 mm to (259.4, 22.4)
- moved S43 0.56 mm to (169.3, 87.0), turned to 8 degrees
- moved SW11 0.56 mm to (230.8, 21.8)
- moved SW20 0.56 mm to (161.7, 49.6)
- moved SW21 0.56 mm to (180.5, 46.9)
- moved SW24 0.56 mm to (238.3, 41.1)
- moved SW25 0.56 mm to (264.4, 41.1)
- moved SW33 0.56 mm to (173.8, 67.1)
- moved SW34 0.56 mm to (192.6, 64.5)
- moved SW37 0.56 mm to (250.4, 60.3)
- moved SW38 0.56 mm to (271.9, 60.3)
- moved SW8 0.56 mm to (173.2, 28.7)
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