File: Libra mini EC.kicad_pcb (KiCad board)
At the start: 2 copper layers, 269.5 x 183.8 mm, 144 parts, among them J1 USB_C_Receptacle_USB2.0_16P, J2 Conn_01x08, J3 Conn_01x18, J4 Conn_01x18, SW1 EC_SW, SW10 EC_SW, SW11 EC_SW, SW12 EC_SW, SW13 EC_SW, SW14 EC_SW, SW15 EC_SW, SW16 EC_SW, SW17 EC_SW, SW18 EC_SW, SW19 EC_SW, SW2 EC_SW, SW20 EC_SW, SW21 EC_SW, SW22 EC_SW, SW23 EC_SW, SW24 EC_SW, SW25 EC_SW, SW26 EC_SW, SW27 EC_SW, SW28 EC_SW, SW29 EC_SW, SW3 EC_SW, SW30 EC_SW, SW31 EC_SW, SW32 EC_SW, SW33 EC_SW, SW34 EC_SW, SW35 EC_SW, SW36 EC_SW, SW37 EC_SW, SW38 EC_SW, SW39 EC_SW, SW4 EC_SW, SW40 EC_SW, SW47 EC_SW, SW5 EC_SW, SW50 EC_SW, SW51 EC_SW, SW52 EC_SW, SW53 EC_SW, SW54 EC_SW, SW55 EC_SW, SW6 EC_SW, SW7 EC_SW, SW8 EC_SW, SW9 EC_SW, U1 STM32G474CBTx, U2 USBLC6-2SC6, U3 TPS7A2033, U4 TPS7A2033, U5 TPS7A2033, U6 OPA2365, U7 4052, U8 OPA2365, U9 4052, Y1 8Mhz 12pF

Commit message: 15.04.2026
Parts:
- removed C20, C22: 1uF, Capacitor_SMD:C_0603_1608Metric
- removed C21, C23: 10uF, Capacitor_SMD:C_0805_2012Metric
- removed U4, U5: TPS7A2033, Package_TO_SOT_SMD:SOT-23-5
- BOOT_SW1, C1, C10, C11, C12, C13, C14, C15, C16, C17, C18, C19, C2, C24, C25, C26, C27, C28, C29, C3, C30, C31, C4, C5, C6, C7, C8, C9, F1, J2, J3, J4, R1, R10, R11, R12, R13, R14, R18, R19, R2, R23, R24, R28, R29, R3, R4, R5, R6, R7, R8, R9, RESET_SW1, U1, U2, U3, Y1: moved to B.Cu
- R15, R16, R17, R20, R21, R22, R25, R26, R27, R30, R31, R32: footprint Capacitor_SMD:C_0805_2012Metric -> Resistor_SMD:R_0805_2012Metric; moved to B.Cu
- moved U7 309.9 mm to (63.5, 72.6), turned to 0 degrees
- moved R17 302.1 mm to (16.3, 29.9), turned to -90 degrees
- moved D4 300.8 mm to (23.8, 69.8)
- moved U6 299.3 mm to (63.5, 79.0), turned to 0 degrees
- moved R22 293.2 mm to (31.4, 23.1), turned to -90 degrees
- moved C26 288.7 mm to (68.7, 81.0), turned to 180 degrees
- moved C24 288.2 mm to (68.7, 75.0)
- moved R13 286.2 mm to (58.7, 83.7), turned to 180 degrees
- moved R14 286.2 mm to (58.7, 86.3), turned to 180 degrees
- moved R18 281.7 mm to (63.1, 83.7), turned to 180 degrees
- moved R19 281.7 mm to (63.1, 86.3), turned to 180 degrees
- moved D3 281.3 mm to (21.8, 31.4)
- moved R16 271.0 mm to (51.2, 21.4), turned to -90 degrees
- moved D2 264.4 mm to (70.2, 32.9)
- moved R21 255.7 mm to (69.8, 24.2), turned to -90 degrees
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Connections:
- SW51 pad 1: COL4 -> COL5
Routing:
- net ROW2: track 0.00 -> 124.5 mm
- net ROW1: track 0.00 -> 121.7 mm
- net ROW0: track 0.00 -> 116.2 mm
- net ROW3: track 0.00 -> 101.5 mm
- net COL3: track 0.00 -> 64.6 mm
- net COL1: track 0.00 -> 63.4 mm
- net COL5: track 0.00 -> 60.3 mm
- net COL0: track 0.00 -> 59.7 mm
- net COL2: track 0.00 -> 43.4 mm
- net COL4: track 0.00 -> 43.4 mm
Other:
- board size 269.5 x 183.8 mm -> 301.7 x 106 mm
