File: Libra mini EC MATRIX.kicad_sch (KiCad schematic)
At the start: 63 parts, among them SW1 EC_SW, SW10 EC_SW, SW11 EC_SW, SW12 EC_SW, SW13 EC_SW, SW14 EC_SW, SW15 EC_SW, SW16 EC_SW, SW17 EC_SW, SW18 EC_SW, SW19 EC_SW, SW2 EC_SW, SW20 EC_SW, SW21 EC_SW, SW22 EC_SW, SW23 EC_SW, SW24 EC_SW, SW25 EC_SW, SW26 EC_SW, SW27 EC_SW, SW28 EC_SW, SW29 EC_SW, SW3 EC_SW, SW30 EC_SW, SW31 EC_SW, SW32 EC_SW, SW33 EC_SW, SW34 EC_SW, SW35 EC_SW, SW36 EC_SW, SW37 EC_SW, SW38 EC_SW, SW39 EC_SW, SW4 EC_SW, SW40 EC_SW, SW41 EC_SW, SW42 EC_SW, SW43 EC_SW, SW44 EC_SW, SW45 EC_SW, SW46 EC_SW, SW47 EC_SW, SW5 EC_SW, SW6 EC_SW, SW7 EC_SW, SW8 EC_SW, SW9 EC_SW

Commit message: 14.04.2026
Parts:
- added SW48: EC_SW, Kicad footprints:ecs_pad_hybrid hotswap_1.25-1_libra_2.286, symbol Kicad symbols:EC_SW
- added SW49, SW50: EC_SW, Kicad footprints:ecs_pad_1U_hybrid_hotswap_V2, symbol Kicad symbols:EC_SW
- SW45: footprint Kicad footprints:ecs_pad_1U_hybrid_hotswap_V2 -> Kicad footprints:ecs_pad_hybrid_hotswap_1.25-1_libra_7.239
- SW46: footprint Kicad footprints:ecs_pad_1U_hybrid_hotswap_V2 -> Kicad footprints:ecs_pad_hybrid_hotswap_1.25-1_libra_2.381
Connections:
- net COL7: now also SW48.1
- net COL8: now also SW49.1
- net COL9: now also SW50.1
- net GND: now also SW48.3 (SG), SW49.3 (SG)
- net ROW3: now also SW48.2, SW49.2, SW50.2
Other:
- moved on the sheet: S43

Commit message: 14.04.2026
Parts:
- removed D13, D14: SK6812MINI, LED_SMD:LED_SK6812MINI_PLCC4_3.5x3.5mm_P1.75mm, symbol LED:SK6812MINI
- added S47: MX_stab, PCM_marbastlib-mx:STAB_MX_2u, symbol PCM_marbastlib-mx:MX_stab
Connections:
- net GND: now also D10.2 (VSS), D11.2 (VSS), D12.2 (VSS), D8.2 (VSS), D9.2 (VSS); no longer D1.2 (VSS), D2.2 (VSS), D3.2 (VSS), D4.2 (VSS), D5.2 (VSS), D6.2 (VSS)
- net RGB: now also D6.1 (DOUT), D7.3 (DIN); no longer D7.1 (DOUT), D8.3 (DIN)
- net RGB_FINISH: now also D12.1 (DOUT)
- net at D8.1 (DOUT): now also D9.3 (DIN)
- new net: D7.1 (DOUT), D8.3 (DIN)
- new net: D1.2 (VSS), D2.2 (VSS), D3.2 (VSS), D4.2 (VSS), D5.2 (VSS), D6.2 (VSS)
Other:
- moved on the sheet: D10, D11, D12, D7, D8, D9
