File: Libra mini EC MATRIX.kicad_sch (KiCad schematic)
At the start: 72 parts, among them SW1 EC_SW, SW10 EC_SW, SW11 EC_SW, SW12 EC_SW, SW13 EC_SW, SW14 EC_SW, SW15 EC_SW, SW16 EC_SW, SW17 EC_SW, SW18 EC_SW, SW19 EC_SW, SW2 EC_SW, SW20 EC_SW, SW21 EC_SW, SW22 EC_SW, SW23 EC_SW, SW24 EC_SW, SW25 EC_SW, SW26 EC_SW, SW27 EC_SW, SW28 EC_SW, SW29 EC_SW, SW3 EC_SW, SW30 EC_SW, SW31 EC_SW, SW32 EC_SW, SW33 EC_SW, SW34 EC_SW, SW35 EC_SW, SW36 EC_SW, SW37 EC_SW, SW38 EC_SW, SW39 EC_SW, SW4 EC_SW, SW40 EC_SW, SW41 EC_SW, SW42 EC_SW, SW43 EC_SW, SW44 EC_SW, SW45 EC_SW, SW46 EC_SW, SW47 EC_SW, SW48 EC_SW, SW49 EC_SW, SW5 EC_SW, SW50 EC_SW, SW51 EC_SW, SW52 EC_SW, SW53 EC_SW, SW54 EC_SW, SW55 EC_SW, SW6 EC_SW, SW7 EC_SW, SW8 EC_SW, SW9 EC_SW

Commit message: 14.04.2026
Parts:
- SW41, SW42, SW43, SW44, SW45, SW46, SW48, SW49: now not fitted; now left out of the parts list
- SW54, SW55: footprint Kicad footprints:ecs_pad_1U_hybrid_hotswap_V2 -> My_footprints:ecs_pad_hybrid_hotswap_1.25-1_libra_2.381
Changed lines of the file:
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@@
 		(unit 1)
 		(exclude_from_sim no)
-		(in_bom yes)
-		(on_board yes)
-		(dnp no)
+		(in_bom no)
+		(on_board no)
+		(dnp yes)
 		(fields_autoplaced yes)
 		(property "Reference" "SW46"
@@
 			)
 		)
-		(property "Footprint" "Kicad footprints:ecs_pad_1U_hybrid_hotswap_V2"
+		(property "Footprint" "My_footprints:ecs_pad_hybrid_hotswap_1.25-1_libra_2.381"
 			(at 201.93 102.87 0)
 			(effects
@@
 		(unit 1)
 		(exclude_from_sim no)
-		(in_bom yes)
-		(on_board yes)
-		(dnp no)
+		(in_bom no)
+		(on_board no)
+		(dnp yes)
 		(fields_autoplaced yes)
 		(property "Reference" "SW49"
@@
 		(unit 1)
 		(exclude_from_sim no)
-		(in_bom yes)
-		(on_board yes)
-		(dnp no)
+		(in_bom no)
+		(on_board no)
+		(dnp yes)
 		(fields_autoplaced yes)
 		(property "Reference" "SW42"
@@
 		(unit 1)
 		(exclude_from_sim no)
-		(in_bom yes)
-		(on_board yes)
-		(dnp no)
+		(in_bom no)
+		(on_board no)
+		(dnp yes)
 		(fields_autoplaced yes)
 		(property "Reference" "SW41"
@@
 		(unit 1)
 		(exclude_from_sim no)
-		(in_bom yes)
-		(on_board yes)
-		(dnp no)
+		(in_bom no)
+		(on_board no)
+		(dnp yes)
 		(fields_autoplaced yes)
 		(property "Reference" "SW43"
@@
 		(unit 1)
 		(exclude_from_sim no)
-		(in_bom yes)
-		(on_board yes)
-		(dnp no)
+		(in_bom no)
+		(on_board no)
+		(dnp yes)
 		(fields_autoplaced yes)
 		(property "Reference" "SW44"
@@
 		(unit 1)
 		(exclude_from_sim no)
-		(in_bom yes)
-		(on_board yes)
-		(dnp no)
+		(in_bom no)
+		(on_board no)
+		(dnp yes)
 		(fields_autoplaced yes)
 		(property "Reference" "SW45"
@@
 			)
 		)
-		(property "Footprint" "Kicad footprints:ecs_pad_1U_hybrid_hotswap_V2"
+		(property "Footprint" "My_footprints:ecs_pad_hybrid_hotswap_1.25-1_libra_2.381"
 			(at 185.42 102.87 0)
 			(effects
@@
 		(unit 1)
 		(exclude_from_sim no)
-		(in_bom yes)
-		(on_board yes)
-		(dnp no)
+		(in_bom no)
+		(on_board no)
+		(dnp yes)
 		(fields_autoplaced yes)
 		(property "Reference" "SW48"

Commit message: 15.04.2026
Connections:
- net COL4: no longer SW42.1, SW51.1
- net COL5: now also SW42.1, SW51.1
Other:
- moved on the sheet: S42, S51, SW42, SW51
Changed lines of the file:
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@@
 	)
 	(junction
+		(at 124.46 92.71)
+		(diameter 0)
+		(color 0 0 0 0)
+	)
+	(junction
 		(at 34.29 57.15)
 		(diameter 0)
@@
 	)
 	(junction
+		(at 116.84 87.63)
+		(diameter 0)
+		(color 0 0 0 0)
+	)
+	(junction
 		(at 234.95 46.99)
 		(diameter 0)
@@
 	)
 	(junction
-		(at 100.33 72.39)
-		(diameter 0)
-		(color 0 0 0 0)
-	)
-	(junction
 		(at 251.46 46.99)
 		(diameter 0)
@@
 	)
 	(junction
-		(at 107.95 92.71)
-		(diameter 0)
-		(color 0 0 0 0)
-	)
-	(junction
 		(at 74.93 77.47)
 		(diameter 0)
@@
 	)
 	(junction
-		(at 100.33 87.63)
+		(at 115.57 78.74)
 		(diameter 0)
 		(color 0 0 0 0)
 	)
 	(junction
-		(at 115.57 78.74)
+		(at 116.84 72.39)
 		(diameter 0)
 		(color 0 0 0 0)
@@
 	)
 	(junction
+		(at 132.08 93.98)
+		(diameter 0)
+		(color 0 0 0 0)
+	)
+	(junction
 		(at 115.57 63.5)
 		(diameter 0)
@@
 	)
 	(junction
-		(at 115.57 93.98)
-		(diameter 0)
-		(color 0 0 0 0)
-	)
-	(junction
 		(at 160.02 63.5)
 		(diameter 0)
@@
 	(wire
 		(pts
+			(xy 132.08 93.98) (xy 160.02 93.98)
+		)
+		(stroke
+			(width 0)
+			(type default)
+		)
+	)
+	(wire
+		(pts
 			(xy 177.8 87.63) (xy 177.8 102.87)
 		)
@@
 	(wire
 		(pts
-			(xy 115.57 93.98) (xy 99.06 93.98)
+			(xy 99.06 93.98) (xy 132.08 93.98)
 		)
 		(stroke
@@
 	(wire
 		(pts
-			(xy 107.95 92.71) (xy 107.95 107.95)
-		)
-		(stroke
-			(width 0)
-			(type default)
-		)
-	)
-	(wire
-		(pts
 			(xy 53.34 173.99) (xy 78.74 173.99)
 		)
@@
 	(wire
 		(pts
-			(xy 160.02 93.98) (xy 160.02 102.87)
+			(xy 116.84 72.39) (xy 116.84 87.63)
 		)
 		(stroke
@@
 	(wire
 		(pts
-			(xy 27.94 173.99) (xy 53.34 173.99)
+			(xy 160.02 93.98) (xy 160.02 102.87)
 		)
 		(stroke
@@
 	(wire
 		(pts
-			(xy 115.57 93.98) (xy 115.57 102.87)
+			(xy 27.94 173.99) (xy 53.34 173.99)
 		)
 		(stroke
@@
 	(wire
 		(pts
+			(xy 132.08 93.98) (xy 132.08 102.87)
+		)
+		(stroke
+			(width 0)
+			(type default)
+		)
+	)
+	(wire
+		(pts
 			(xy 99.06 78.74) (xy 82.55 78.74)
 		)
@@
 	(wire
 		(pts
-			(xy 107.95 92.71) (xy 139.7 92.71)
+			(xy 91.44 92.71) (xy 124.46 92.71)
 		)
 		(stroke
@@
 	(wire
 		(pts
-			(xy 201.93 46.99) (xy 218.44 46.99)
+			(xy 116.84 87.63) (xy 116.84 102.87)
 		)
 		(stroke
@@
 	(wire
 		(pts
-			(xy 82.55 48.26) (xy 66.04 48.26)
+			(xy 201.93 46.99) (xy 218.44 46.99)
 		)
 		(stroke
@@
 	(wire
 		(pts
-			(xy 115.57 87.63) (xy 115.57 93.98)
+			(xy 82.55 48.26) (xy 66.04 48.26)
 		)
 		(stroke
@@
 	(wire
 		(pts
-			(xy 115.57 93.98) (xy 160.02 93.98)
-		)
-		(stroke
-			(width 0)
-			(type default)
-		)
-	)
-	(wire
-		(pts
 			(xy 66.04 48.26) (xy 49.53 48.26)
 		)
@@
 	(wire
 		(pts
+			(xy 124.46 92.71) (xy 124.46 107.95)
+		)
+		(stroke
+			(width 0)
+			(type default)
+		)
+	)
+	(wire
+		(pts
 			(xy 218.44 62.23) (xy 234.95 62.23)
 		)
@@
 	(wire
 		(pts
+			(xy 124.46 92.71) (xy 139.7 92.71)
+		)
+		(stroke
+			(width 0)
+			(type default)
+		)
+	)
+	(wire
+		(pts
 			(xy 177.8 41.91) (xy 177.8 57.15)
 		)
@@
 	(wire
 		(pts
-			(xy 91.44 92.71) (xy 107.95 92.71)
-		)
-		(stroke
-			(width 0)
-			(type default)
-		)
-	)
-	(wire
-		(pts
 			(xy 41.91 62.23) (xy 58.42 62.23)
 		)
@@
 	(wire
 		(pts
-			(xy 100.33 72.39) (xy 100.33 87.63)
+			(xy 132.08 87.63) (xy 132.08 93.98)
 		)
 		(stroke
@@
 	(wire
 		(pts
-			(xy 100.33 87.63) (xy 100.33 102.87)
-		)
-		(stroke
-			(width 0)
-			(type default)
-		)
-	)
-	(wire
-		(pts
 			(xy 86.36 157.48) (xy 96.52 157.48)
 		)
@@
 	(symbol
 		(lib_id "Kicad symbols:EC_SW")
-		(at 107.95 102.87 0)
+		(at 124.46 102.87 0)
 		(unit 1)
 		(exclude_from_sim no)
@@
 		(fields_autoplaced yes)
 		(property "Reference" "SW51"
-			(at 107.95 95.25 0)
+			(at 124.46 95.25 0)
 			(effects
 				(font
@@
 		)
 		(property "Value" "EC_SW"
-			(at 107.95 97.79 0)
+			(at 124.46 97.79 0)
 			(effects
 				(font
@@
 		)
 		(property "Footprint" "Kicad footprints:ecs_pad_hybrid_hotswap_1.25-1_libra_2.381"
-			(at 107.95 102.87 0)
+			(at 124.46 102.87 0)
 			(effects
 				(font
@@
 		)
 		(property "Datasheet" ""
-			(at 107.95 102.87 0)
+			(at 124.46 102.87 0)
 			(effects
 				(font
@@
 		)
 		(property "Description" ""
-			(at 107.95 102.87 0)
+			(at 124.46 102.87 0)
 			(effects
 				(font
@@
 	(symbol
 		(lib_id "Kicad symbols:EC_SW")
-		(at 107.95 87.63 0)
+		(at 124.46 87.63 0)
 		(unit 1)
 		(exclude_from_sim no)
@@
 		(fields_autoplaced yes)
 		(property "Reference" "SW42"
-			(at 107.95 80.01 0)
+			(at 124.46 80.01 0)
 			(effects
 				(font
@@
 		)
 		(property "Value" "EC_SW"
-			(at 107.95 82.55 0)
+			(at 124.46 82.55 0)
 			(effects
 				(font
@@
 		)
 		(property "Footprint" "Kicad footprints:ecs_pad_1U_hybrid_hotswap_V2"
-			(at 107.95 87.63 0)
+			(at 124.46 87.63 0)
 			(effects
 				(font
@@
 		)
 		(property "Datasheet" ""
-			(at 107.95 87.63 0)
+			(at 124.46 87.63 0)
 			(effects
 				(font
@@
 		)
 		(property "Description" ""
-			(at 107.95 87.63 0)
+			(at 124.46 87.63 0)
 			(effects
 				(font
@@
 	(symbol
 		(lib_id "PCM_marbastlib-mx:MX_stab")
-		(at 107.95 114.3 0)
+		(at 132.08 115.57 0)
 		(unit 1)
 		(exclude_from_sim no)
@@
 		(fields_autoplaced yes)
 		(property "Reference" "S42"
-			(at 114.3 112.9029 0)
+			(at 138.43 114.1729 0)
 			(effects
 				(font
@@
 		)
 		(property "Value" "MX_stab"
-			(at 114.3 115.4429 0)
+			(at 138.43 116.7129 0)
 			(effects
 				(font
@@
 		)
 		(property "Footprint" "PCM_marbastlib-mx:STAB_MX_2u"
-			(at 107.95 114.3 0)
+			(at 132.08 115.57 0)
 			(effects
 				(font
@@
 		)
 		(property "Datasheet" ""
-			(at 107.95 114.3 0)
+			(at 132.08 115.57 0)
 			(effects
 				(font
@@
 		)
 		(property "Description" "Cherry MX-style stabilizer"
-			(at 107.95 114.3 0)
+			(at 132.08 115.57 0)
 			(effects
 				(font
@@
 	(symbol
 		(lib_id "PCM_marbastlib-mx:MX_stab")
-		(at 107.95 129.54 0)
+		(at 132.08 130.81 0)
 		(unit 1)
 		(exclude_from_sim no)
@@
 		(fields_autoplaced yes)
 		(property "Reference" "S51"
-			(at 114.3 128.1429 0)
+			(at 138.43 129.4129 0)
 			(effects
 				(font
@@
 		)
 		(property "Value" "MX_stab"
-			(at 114.3 130.6829 0)
+			(at 138.43 131.9529 0)
 			(effects
 				(font
@@
 		)
 		(property "Footprint" "PCM_marbastlib-mx:STAB_MX_2.25u"
-			(at 107.95 129.54 0)
+			(at 132.08 130.81 0)
 			(effects
 				(font
@@
 		)
 		(property "Datasheet" ""
-			(at 107.95 129.54 0)
+			(at 132.08 130.81 0)
 			(effects
 				(font
@@
 		)
 		(property "Description" "Cherry MX-style stabilizer"
-			(at 107.95 129.54 0)
+			(at 132.08 130.81 0)
 			(effects
 				(font
