File: Libra mini EC.kicad_sch (KiCad schematic)
At the start: 48 parts, among them J1 USB_C_Receptacle_USB2.0_16P, J2 Conn_01x08, J3 Conn_01x18, J4 Conn_01x18, U1 STM32G474CBTx, U2 USBLC6-2SC6, U3 TPS7A2033, U4 TPS7A2033, U5 TPS7A2033, Y1 8Mhz 12pF

Commit message: 15.04.2026
Parts:
- removed C20, C22: 1uF, Capacitor_SMD:C_0603_1608Metric, symbol Device:C_Small
- removed C21, C23: 10uF, Capacitor_SMD:C_0805_2012Metric, symbol Device:C_Small
- removed U4, U5: TPS7A2033, Package_TO_SOT_SMD:SOT-23-5, symbol Regulator_Linear:TLV75533PDBV
- C11, C12, C13, C14: now not fitted
