File: Delta EC MATRIX.kicad_sch (KiCad schematic)
At the start: 72 parts, among them SW1 EC_SW, SW10 EC_SW, SW11 EC_SW, SW12 EC_SW, SW13 EC_SW, SW14 EC_SW, SW15 EC_SW, SW16 EC_SW, SW17 EC_SW, SW18 EC_SW, SW19 EC_SW, SW2 EC_SW, SW20 EC_SW, SW21 EC_SW, SW22 EC_SW, SW23 EC_SW, SW24 EC_SW, SW25 EC_SW, SW26 EC_SW, SW27 EC_SW, SW28 EC_SW, SW29 EC_SW, SW3 EC_SW, SW30 EC_SW, SW31 EC_SW, SW32 EC_SW, SW33 EC_SW, SW34 EC_SW, SW35 EC_SW, SW36 EC_SW, SW37 EC_SW, SW38 EC_SW, SW39 EC_SW, SW4 EC_SW, SW40 EC_SW, SW41 EC_SW, SW42 EC_SW, SW43 EC_SW, SW44 EC_SW, SW45 EC_SW, SW46 EC_SW, SW47 EC_SW, SW48 EC_SW, SW49 EC_SW, SW5 EC_SW, SW50 EC_SW, SW51 EC_SW, SW52 EC_SW, SW53 EC_SW, SW54 EC_SW, SW55 EC_SW, SW6 EC_SW, SW7 EC_SW, SW8 EC_SW, SW9 EC_SW

Commit message: 16.04.2026
Parts:
- SW25, SW32, SW33, SW34, SW35, SW36: footprint Kicad footprints:ecs_pad_1U_hybrid_hotswap_V2 -> Kicad footprints:ecs_pad_1U_hybrid_hotswap_V2_switched_sides
- SW39, SW40, SW50, SW51, SW52, SW53: footprint Kicad footprints:ecs_pad_hybrid_hotswap_1.25-1_libra_2.381 -> Kicad footprints:ecs_pad_hybrid_hotswap_2.381_V2
- SW54, SW55: footprint My_footprints:ecs_pad_hybrid_hotswap_1.25-1_libra_2.381 -> Kicad footprints:ecs_pad_hybrid_hotswap_2.381_V2
Changed lines of the file:
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@@
 			)
 		)
-		(property "Footprint" "My_footprints:ecs_pad_hybrid_hotswap_1.25-1_libra_2.381"
+		(property "Footprint" "Kicad footprints:ecs_pad_hybrid_hotswap_2.381_V2"
 			(at 201.93 102.87 0)
 			(effects
@@
 			)
 		)
-		(property "Footprint" "Kicad footprints:ecs_pad_hybrid_hotswap_1.25-1_libra_2.381"
+		(property "Footprint" "Kicad footprints:ecs_pad_hybrid_hotswap_2.381_V2"
 			(at 58.42 87.63 0)
 			(effects
@@
 			)
 		)
-		(property "Footprint" "Kicad footprints:ecs_pad_1U_hybrid_hotswap_V2"
+		(property "Footprint" "Kicad footprints:ecs_pad_1U_hybrid_hotswap_V2_switched_sides"
 			(at 234.95 57.15 0)
 			(effects
@@
 			)
 		)
-		(property "Footprint" "Kicad footprints:ecs_pad_hybrid_hotswap_1.25-1_libra_2.381"
+		(property "Footprint" "Kicad footprints:ecs_pad_hybrid_hotswap_2.381_V2"
 			(at 124.46 102.87 0)
 			(effects
@@
 			)
 		)
-		(property "Footprint" "Kicad footprints:ecs_pad_1U_hybrid_hotswap_V2"
+		(property "Footprint" "Kicad footprints:ecs_pad_1U_hybrid_hotswap_V2_switched_sides"
 			(at 152.4 72.39 0)
 			(effects
@@
 			)
 		)
-		(property "Footprint" "Kicad footprints:ecs_pad_hybrid_hotswap_1.25-1_libra_2.381"
+		(property "Footprint" "Kicad footprints:ecs_pad_hybrid_hotswap_2.381_V2"
 			(at 91.44 102.87 0)
 			(effects
@@
 			)
 		)
-		(property "Footprint" "Kicad footprints:ecs_pad_1U_hybrid_hotswap_V2"
+		(property "Footprint" "Kicad footprints:ecs_pad_1U_hybrid_hotswap_V2_switched_sides"
 			(at 168.91 72.39 0)
 			(effects
@@
 			)
 		)
-		(property "Footprint" "Kicad footprints:ecs_pad_hybrid_hotswap_1.25-1_libra_2.381"
+		(property "Footprint" "Kicad footprints:ecs_pad_hybrid_hotswap_2.381_V2"
 			(at 168.91 102.87 0)
 			(effects
@@
 			)
 		)
-		(property "Footprint" "Kicad footprints:ecs_pad_1U_hybrid_hotswap_V2"
+		(property "Footprint" "Kicad footprints:ecs_pad_1U_hybrid_hotswap_V2_switched_sides"
 			(at 201.93 72.39 0)
 			(effects
@@
 			)
 		)
-		(property "Footprint" "Kicad footprints:ecs_pad_1U_hybrid_hotswap_V2"
+		(property "Footprint" "Kicad footprints:ecs_pad_1U_hybrid_hotswap_V2_switched_sides"
 			(at 218.44 72.39 0)
 			(effects
@@
 			)
 		)
-		(property "Footprint" "My_footprints:ecs_pad_hybrid_hotswap_1.25-1_libra_2.381"
+		(property "Footprint" "Kicad footprints:ecs_pad_hybrid_hotswap_2.381_V2"
 			(at 185.42 102.87 0)
 			(effects
@@
 			)
 		)
-		(property "Footprint" "Kicad footprints:ecs_pad_1U_hybrid_hotswap_V2"
+		(property "Footprint" "Kicad footprints:ecs_pad_1U_hybrid_hotswap_V2_switched_sides"
 			(at 185.42 72.39 0)
 			(effects
@@
 			)
 		)
-		(property "Footprint" "Kicad footprints:ecs_pad_hybrid_hotswap_1.25-1_libra_2.381"
+		(property "Footprint" "Kicad footprints:ecs_pad_hybrid_hotswap_2.381_V2"
 			(at 152.4 102.87 0)
 			(effects
@@
 			)
 		)
-		(property "Footprint" "Kicad footprints:ecs_pad_hybrid_hotswap_1.25-1_libra_2.381"
+		(property "Footprint" "Kicad footprints:ecs_pad_hybrid_hotswap_2.381_V2"
 			(at 41.91 87.63 0)
 			(effects
