File: Delta EC MATRIX.kicad_sch (KiCad schematic)
At the start: 72 parts, among them SW1 EC_SW, SW10 EC_SW, SW11 EC_SW, SW12 EC_SW, SW13 EC_SW, SW14 EC_SW, SW15 EC_SW, SW16 EC_SW, SW17 EC_SW, SW18 EC_SW, SW19 EC_SW, SW2 EC_SW, SW20 EC_SW, SW21 EC_SW, SW22 EC_SW, SW23 EC_SW, SW24 EC_SW, SW25 EC_SW, SW26 EC_SW, SW27 EC_SW, SW28 EC_SW, SW29 EC_SW, SW3 EC_SW, SW30 EC_SW, SW31 EC_SW, SW32 EC_SW, SW33 EC_SW, SW34 EC_SW, SW35 EC_SW, SW36 EC_SW, SW37 EC_SW, SW38 EC_SW, SW39 EC_SW, SW4 EC_SW, SW40 EC_SW, SW41 EC_SW, SW42 EC_SW, SW43 EC_SW, SW44 EC_SW, SW45 EC_SW, SW46 EC_SW, SW47 EC_SW, SW48 EC_SW, SW49 EC_SW, SW5 EC_SW, SW50 EC_SW, SW51 EC_SW, SW52 EC_SW, SW53 EC_SW, SW54 EC_SW, SW55 EC_SW, SW6 EC_SW, SW7 EC_SW, SW8 EC_SW, SW9 EC_SW

Commit message: 17.04.2026
Connections:
- net COL4: now also SW42.1, SW51.1
- net COL5: no longer SW42.1, SW51.1
Other:
- moved on the sheet: SW42, SW51
Changed lines of the file:
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@@
 	)
 	(junction
-		(at 124.46 92.71)
+		(at 107.95 92.71)
 		(diameter 0)
 		(color 0 0 0 0)
@@
 	)
 	(junction
-		(at 116.84 87.63)
-		(diameter 0)
-		(color 0 0 0 0)
-	)
-	(junction
 		(at 234.95 46.99)
 		(diameter 0)
@@
 	)
 	(junction
+		(at 100.33 87.63)
+		(diameter 0)
+		(color 0 0 0 0)
+	)
+	(junction
 		(at 91.44 92.71)
 		(diameter 0)
@@
 	)
 	(junction
-		(at 116.84 72.39)
-		(diameter 0)
-		(color 0 0 0 0)
-	)
-	(junction
 		(at 58.42 77.47)
 		(diameter 0)
@@
 	)
 	(junction
-		(at 132.08 93.98)
+		(at 115.57 93.98)
 		(diameter 0)
 		(color 0 0 0 0)
@@
 	)
 	(junction
+		(at 100.33 72.39)
+		(diameter 0)
+		(color 0 0 0 0)
+	)
+	(junction
 		(at 82.55 48.26)
 		(diameter 0)
@@
 	(wire
 		(pts
-			(xy 132.08 93.98) (xy 160.02 93.98)
+			(xy 115.57 93.98) (xy 160.02 93.98)
 		)
 		(stroke
@@
 	(wire
 		(pts
-			(xy 99.06 93.98) (xy 132.08 93.98)
+			(xy 99.06 93.98) (xy 115.57 93.98)
 		)
 		(stroke
@@
 	(wire
 		(pts
-			(xy 116.84 72.39) (xy 116.84 87.63)
-		)
-		(stroke
-			(width 0)
-			(type default)
-		)
-	)
-	(wire
-		(pts
 			(xy 160.02 93.98) (xy 160.02 102.87)
 		)
@@
 	(wire
 		(pts
-			(xy 132.08 93.98) (xy 132.08 102.87)
+			(xy 115.57 93.98) (xy 115.57 102.87)
 		)
 		(stroke
@@
 	(wire
 		(pts
-			(xy 91.44 92.71) (xy 124.46 92.71)
+			(xy 91.44 92.71) (xy 107.95 92.71)
 		)
 		(stroke
@@
 	(wire
 		(pts
-			(xy 116.84 87.63) (xy 116.84 102.87)
+			(xy 100.33 87.63) (xy 100.33 102.87)
 		)
 		(stroke
@@
 	(wire
 		(pts
-			(xy 124.46 92.71) (xy 124.46 107.95)
+			(xy 107.95 92.71) (xy 107.95 107.95)
 		)
 		(stroke
@@
 	(wire
 		(pts
-			(xy 124.46 92.71) (xy 139.7 92.71)
+			(xy 107.95 92.71) (xy 139.7 92.71)
 		)
 		(stroke
@@
 	(wire
 		(pts
+			(xy 100.33 72.39) (xy 100.33 87.63)
+		)
+		(stroke
+			(width 0)
+			(type default)
+		)
+	)
+	(wire
+		(pts
 			(xy 27.94 148.59) (xy 27.94 149.86)
 		)
@@
 	(wire
 		(pts
-			(xy 132.08 87.63) (xy 132.08 93.98)
+			(xy 115.57 87.63) (xy 115.57 93.98)
 		)
 		(stroke
@@
 	(symbol
 		(lib_id "Kicad symbols:EC_SW")
-		(at 124.46 102.87 0)
+		(at 107.95 102.87 0)
 		(unit 1)
 		(exclude_from_sim no)
@@
 		(fields_autoplaced yes)
 		(property "Reference" "SW51"
-			(at 124.46 95.25 0)
+			(at 107.95 95.25 0)
 			(effects
 				(font
@@
 		)
 		(property "Value" "EC_SW"
-			(at 124.46 97.79 0)
+			(at 107.95 97.79 0)
 			(effects
 				(font
@@
 		)
 		(property "Footprint" "Kicad footprints:ecs_pad_hybrid_hotswap_2.381_V2"
-			(at 124.46 102.87 0)
+			(at 107.95 102.87 0)
 			(effects
 				(font
@@
 		)
 		(property "Datasheet" ""
-			(at 124.46 102.87 0)
+			(at 107.95 102.87 0)
 			(effects
 				(font
@@
 		)
 		(property "Description" ""
-			(at 124.46 102.87 0)
+			(at 107.95 102.87 0)
 			(effects
 				(font
@@
 	(symbol
 		(lib_id "Kicad symbols:EC_SW")
-		(at 124.46 87.63 0)
+		(at 107.95 87.63 0)
 		(unit 1)
 		(exclude_from_sim no)
@@
 		(fields_autoplaced yes)
 		(property "Reference" "SW42"
-			(at 124.46 80.01 0)
+			(at 107.95 80.01 0)
 			(effects
 				(font
@@
 		)
 		(property "Value" "EC_SW"
-			(at 124.46 82.55 0)
+			(at 107.95 82.55 0)
 			(effects
 				(font
@@
 		)
 		(property "Footprint" "Kicad footprints:ecs_pad_1U_hybrid_hotswap_V2"
-			(at 124.46 87.63 0)
+			(at 107.95 87.63 0)
 			(effects
 				(font
@@
 		)
 		(property "Datasheet" ""
-			(at 124.46 87.63 0)
+			(at 107.95 87.63 0)
 			(effects
 				(font
@@
 		)
 		(property "Description" ""
-			(at 124.46 87.63 0)
+			(at 107.95 87.63 0)
 			(effects
 				(font
