File: Delta EC.kicad_pcb (KiCad board)
At the start: 2 copper layers, 301.7 x 106 mm, 138 parts, among them J1 USB_C_Receptacle_USB2.0_16P, J2 Conn_01x08, J3 Conn_01x18, J4 Conn_01x18, SW1 EC_SW, SW10 EC_SW, SW11 EC_SW, SW12 EC_SW, SW13 EC_SW, SW14 EC_SW, SW15 EC_SW, SW16 EC_SW, SW17 EC_SW, SW18 EC_SW, SW19 EC_SW, SW2 EC_SW, SW20 EC_SW, SW21 EC_SW, SW22 EC_SW, SW23 EC_SW, SW24 EC_SW, SW25 EC_SW, SW26 EC_SW, SW27 EC_SW, SW28 EC_SW, SW29 EC_SW, SW3 EC_SW, SW30 EC_SW, SW31 EC_SW, SW32 EC_SW, SW33 EC_SW, SW34 EC_SW, SW35 EC_SW, SW36 EC_SW, SW37 EC_SW, SW38 EC_SW, SW39 EC_SW, SW4 EC_SW, SW40 EC_SW, SW47 EC_SW, SW5 EC_SW, SW50 EC_SW, SW51 EC_SW, SW52 EC_SW, SW53 EC_SW, SW54 EC_SW, SW55 EC_SW, SW6 EC_SW, SW7 EC_SW, SW8 EC_SW, SW9 EC_SW, U1 STM32G474CBTx, U2 USBLC6-2SC6, U3 TPS7A2033, U6 OPA2365, U7 4052, U8 OPA2365, U9 4052, Y1 8Mhz 12pF

Commit message: 16.04.2026
Connections:
- U1 pad 37: unconnected-(U1-PA13-Pad37) -> SWDIO
- U1 pad 38: unconnected-(U1-PA14-Pad38) -> SWCLK
- U1 pad 40: MUX_S0 -> SWO
- U1 pad 41: MUX_S1 -> MUX_S0
- U1 pad 42: MUX0_EN -> MUX_S1
- U1 pad 43: MUX1_EN -> MUX0_EN
- U1 pad 44: unconnected-(U1-PB7-Pad44) -> MUX1_EN

Commit message: 16.04.2026
Parts:
- added J5: JSB USB, Connector_JST:JST_SH_SM04B-SRSS-TB_1x04-1MP_P1.00mm_Horizontal, B.Cu at (248.8, 41.3)
- J2: value Conn_01x08 -> SOICbite
- J3: value Conn_01x18 -> FFC Daughter side
- J4: value Conn_01x18 -> FFC Main side
- SW25, SW32, SW33, SW34, SW35, SW36: footprint Kicad footprints:ecs_pad_1U_hybrid_hotswap_V2 -> Kicad footprints:ecs_pad_1U_hybrid_hotswap_V2_switched_sides
- SW39, SW40, SW50, SW51, SW52, SW53: footprint Kicad footprints:ecs_pad_hybrid_hotswap_1.25-1_libra_2.381 -> Kicad footprints:ecs_pad_hybrid_hotswap_2.381_V2
- SW54, SW55: footprint My_footprints:ecs_pad_hybrid_hotswap_1.25-1_libra_2.381 -> Kicad footprints:ecs_pad_hybrid_hotswap_2.381_V2
- moved C17 55.4 mm to (220.3, 72.0)
- moved C18 54.7 mm to (216.7, 71.8), turned to -90 degrees
- moved R11 54.3 mm to (218.7, 72.0), turned to -90 degrees
- moved D8 23.6 mm to (221.9, 52.8)
- moved R30 19.0 mm to (271.9, 50.4)
- moved D10 16.6 mm to (238.1, 29.8)
- moved R27 8.20 mm to (155.2, 40.9)
- moved C3 8.04 mm to (231.0, 73.0), turned to 180 degrees
- moved C1 7.17 mm to (231.8, 82.9), turned to 180 degrees
- moved C5 6.78 mm to (231.5, 81.5), turned to 180 degrees
- moved C8 6.38 mm to (218.3, 75.4), turned to -90 degrees
- moved C4 5.32 mm to (229.1, 83.5), turned to 0 degrees
- moved D11 5.17 mm to (198.0, 34.1)
- moved C7 4.90 mm to (219.6, 75.8), turned to -90 degrees
- moved C2 4.86 mm to (221.9, 73.4), turned to -90 degrees
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Connections:
- J2 pad 5: RESET -> SWO
- J2 pad 6: SWDIO -> SWCLK
- J2 pad 7: SWCLK -> SWDIO
- J2 pad 8: SWO -> RESET
- J3 pad 10: GND -> DISCHARGE0
- J3 pad 11: MUX_S1 -> MUX_S0
- J3 pad 12: MUX_S0 -> MUX_S1
- J3 pad 3: DISCHARGE1 -> +3.3V
- J3 pad 4: GND -> DISCHARGE1
- J3 pad 5: ADC1_IN -> GND
- J3 pad 6: GND -> ADC1_IN
- J3 pad 7: DISCHARGE0 -> GND
- J3 pad 8: GND -> ADC0_IN
- J3 pad 9: ADC0_IN -> GND
- J4 pad 10: ADC2_IN -> GND
- J4 pad 11: GND -> ADC0_IN
- J4 pad 12: DISCHARGE2 -> GND
- J4 pad 13: GND -> ADC1_IN
- J4 pad 14: ADC3_IN -> GND
- J4 pad 15: GND -> DISCHARGE1
- J4 pad 16: DISCHARGE3 -> +3.3V
- J4 pad 6: MUX1_EN -> MUX0_EN
- J4 pad 9: GND -> DISCHARGE0
Routing:
- net ROW2: track 124.5 -> 270.9 mm
- net ROW1: track 121.7 -> 246.3 mm
- net ROW0: track 116.2 -> 224.8 mm
- net COL7: track 0.00 -> 68.0 mm
- net COL6: track 0.00 -> 61.2 mm
- net COL11: track 0.00 -> 59.9 mm
- net ROW3: track 101.5 -> 52.9 mm
- net COL10: track 0.00 -> 46.9 mm
- net COL9: track 0.00 -> 38.7 mm
- net COL8: track 0.00 -> 38.7 mm
- net +3.3V: track 0.00 -> 21.7 mm, vias 0 -> 4
- net SWDIO: track 0.00 -> 12.7 mm, vias 0 -> 1
- net SWCLK: track 0.00 -> 11.5 mm, vias 0 -> 1
- net SWO: track 0.00 -> 10.1 mm, vias 0 -> 1
- net RESET: track 0.00 -> 7.04 mm, vias 0 -> 1
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