File: Delta EC.kicad_pcb (KiCad board)
At the start: 2 copper layers, 301.7 x 106 mm, 139 parts, among them J1 USB_C_Receptacle_USB2.0_16P, J2 SOICbite, J3 FFC Daughter side, J4 FFC Main side, J5 JSB USB, SW1 EC_SW, SW10 EC_SW, SW11 EC_SW, SW12 EC_SW, SW13 EC_SW, SW14 EC_SW, SW15 EC_SW, SW16 EC_SW, SW17 EC_SW, SW18 EC_SW, SW19 EC_SW, SW2 EC_SW, SW20 EC_SW, SW21 EC_SW, SW22 EC_SW, SW23 EC_SW, SW24 EC_SW, SW25 EC_SW, SW26 EC_SW, SW27 EC_SW, SW28 EC_SW, SW29 EC_SW, SW3 EC_SW, SW30 EC_SW, SW31 EC_SW, SW32 EC_SW, SW33 EC_SW, SW34 EC_SW, SW35 EC_SW, SW36 EC_SW, SW37 EC_SW, SW38 EC_SW, SW39 EC_SW, SW4 EC_SW, SW40 EC_SW, SW47 EC_SW, SW5 EC_SW, SW50 EC_SW, SW51 EC_SW, SW52 EC_SW, SW53 EC_SW, SW54 EC_SW, SW55 EC_SW, SW6 EC_SW, SW7 EC_SW, SW8 EC_SW, SW9 EC_SW, U1 STM32G474CBTx, U2 USBLC6-2SC6, U3 TPS7A2033, U6 OPA2365, U7 4052, U8 OPA2365, U9 4052, Y1 8Mhz 12pF

Commit message: 17.04.2026
Parts:
- J3, J4: footprint Connector_FFC-FPC:JUSHUO_AFA07-S18FCA-00_1x18-1MP_P1.0mm_Horizontal -> Connector_FFC-FPC:Amphenol_F32Q-1A7x1-11018_1x18-1MP_P0.5mm_Horizontal
- moved J4 109.4 mm to (70.4, 79.6), turned to -90 degrees
- moved D5 18.7 mm to (96.4, 84.1)
- moved C24 15.7 mm to (55.4, 66.5)
- moved D4 10.1 mm to (32.5, 75.0)
- moved C26 9.11 mm to (64.8, 72.7)
- moved U7 6.26 mm to (57.9, 69.9), turned to 180 degrees
- moved SW51 2.38 mm to (112.2, 87.1), turned to -8 degrees
- moved U6 2.19 mm to (62.4, 77.1), turned to 90 degrees
Connections:
- J4 pad 1: RGB -> RGB_START
- J4 pad 10: GND -> DISCHARGE0
- J4 pad 11: ADC0_IN -> MUX_S1
- J4 pad 12: GND -> MUX_S0
- J4 pad 13: ADC1_IN -> MUX0_EN
- J4 pad 14: GND -> ROW3
- J4 pad 15: DISCHARGE1 -> ROW2
- J4 pad 16: +3.3V -> ROW1
- J4 pad 17: +5V -> ROW0
- J4 pad 18: RGB_START -> RGB
- J4 pad 2: ROW0 -> +5V
- J4 pad 3: ROW1 -> +3.3V
- J4 pad 4: ROW2 -> DISCHARGE1
- J4 pad 5: ROW3 -> GND
- J4 pad 6: MUX0_EN -> ADC1_IN
- J4 pad 7: MUX_S1 -> GND
- J4 pad 8: MUX_S0 -> ADC0_IN
- J4 pad 9: DISCHARGE0 -> GND
- SW51 pad 1: COL5 -> COL4
Routing:
- net ROW2: track 270.9 -> 0.00 mm
- net ROW1: track 246.3 -> 0.00 mm
- net ROW0: track 224.8 -> 0.00 mm
- net COL1: track 63.4 -> 17.8 mm
- net COL3: track 64.6 -> 29.4 mm
- net ROW3: track 52.9 -> 23.5 mm
- net COL2: track 43.4 -> 14.5 mm
- net COL4: track 43.4 -> 64.8 mm
- net COL0: track 59.7 -> 42.7 mm
- net COL5: track 60.3 -> 45.0 mm
- net DISCHARGE0: track 0.00 -> 14.3 mm
- net SWDIO: track 12.7 -> 3.45 mm
- net SWCLK: track 11.5 -> 2.62 mm
- net SWO: track 10.1 -> 1.57 mm
- net DISCHARGE1: track 0.00 -> 7.84 mm
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